File: blackBoxProbe.sch (KiCad schematic (older format))
At the start: 82 parts, among them J1 USB-ID, J2 JTAG_2X05, J3 JTAG_2X05, J4 Conn_01x04, Q1 Q_NMOS_DUAL, Q2 Q_PMOS_DUAL, U1 MCP1702-MB, U2 USBLC6-2, U3 STM32F103CBT, U4 74X2T45, U5 74X2T45, U6 74X2T45, U7 74X2T45, Y1 8.000MHz

Commit message: minor silkscreen updates
Parts:
- N2: value V20180715 -> V20180716
Changed lines of the file:
@@
 P 850 7700
 F 0 "N2" H 850 7800 60  0000 C CNN
-F 1 "V20180715" H 850 7700 60  0000 C CNN
+F 1 "V20180716" H 850 7700 60  0000 C CNN
 F 2 "SquantorLabels:Label_version" H 850 7700 60  0001 C CNN
 F 3 "" H 850 7700 60  0001 C CNN

Commit message: converted to kicad 5 and some modifications
Parts:
- added R? (x2): 10K, SquantorRcl:R_0603_hand, symbol Device:R
- C1, C10, C11, C12, C13, C14, C15, C16, C17, C18, C19, C2, C20, C21, C22, C3, C4, C5, C6, C7, C8, C9: symbol C -> Device:C
- D1, D2, D3, D4: symbol LED -> Device:LED
- H1, H2: symbol Drill_Hole_no_metal -> SquantorPCBOutline:Drill_Hole_no_metal
- J1: symbol USB-ID -> SquantorUsb:USB-ID
- J2, J3: symbol JTAG_2X05 -> SquantorConnectors:JTAG_2X05
- J4: symbol Conn_01x04 -> Connector_Generic:Conn_01x04
- N1: symbol OHWLOGO -> SquantorLabels:OHWLOGO
- N2: value V20180716 -> V20180728; symbol VYYYYMMDD -> SquantorLabels:VYYYYMMDD
- N3: symbol VYYYYMMDD -> SquantorLabels:VYYYYMMDD
- Q1: symbol Q_NMOS_DUAL -> SquantorDevice:Q_NMOS_DUAL
- Q2: symbol Q_PMOS_DUAL -> SquantorDevice:Q_PMOS_DUAL
- R1, R10, R11, R12, R13, R14, R15, R16, R17, R18, R19, R2, R20, R21, R22, R23, R24, R25, R26, R27, R28, R29, R3, R30, R31, R32, R33, R34, R35, R36, R4, R5, R6, R7, R8, R9: symbol R -> Device:R
- S1: symbol 2pin_tact_switch -> SquantorButtons:2pin_tact_switch
- U1: symbol MCP1702-MB -> SquantorMicrochip:MCP1702-MB
- U2: footprint TO_SOT_Packages_SMD:SOT-23-6_Handsoldering -> SquantorIC:SOT23-6-HAND; symbol USBLC6-2 -> SquantorST:USBLC6-2
- U3: symbol STM32F103CBT -> SquantorST:STM32F103CBT
- U4, U5, U6, U7: symbol 74X2T45 -> SquantorLogic:74X2T45
- Y1: symbol Crystal -> Device:Crystal
Connections:
- net +3V3: now also R?.1
- net GND: now also R?.1
- net MCU_TCK: now also R?.2
- net MCU_TMS: now also R?.2

Commit message: updates
Parts:
- gave numbers to parts that had none: 2
Changed lines of the file:
@@
 	3900 5150 3950 5150
 $Comp
-L Device:R R?
+L Device:R R38
 U 1 1 5B624833
 P 3200 6800
-F 0 "R?" V 3280 6800 50  0000 C CNN
+F 0 "R38" V 3280 6800 50  0000 C CNN
 F 1 "10K" V 3200 6800 50  0000 C CNN
 F 2 "SquantorRcl:R_0603_hand" V 3130 6800 50  0001 C CNN
@@
 $EndComp
 $Comp
-L power:GND #PWR?
+L power:GND #PWR0101
 U 1 1 5B624A06
 P 3400 6800
-F 0 "#PWR?" H 3400 6550 50  0001 C CNN
+F 0 "#PWR0101" H 3400 6550 50  0001 C CNN
 F 1 "GND" H 3400 6650 50  0000 C CNN
 F 2 "" H 3400 6800 50  0001 C CNN
@@
 MCU_TCK
 $Comp
-L Device:R R?
+L Device:R R37
 U 1 1 5B6755F6
 P 2950 6700
-F 0 "R?" V 3030 6700 50  0000 C CNN
+F 0 "R37" V 3030 6700 50  0000 C CNN
 F 1 "10K" V 2950 6700 50  0000 C CNN
 F 2 "SquantorRcl:R_0603_hand" V 2880 6700 50  0001 C CNN
@@
 $EndComp
 $Comp
-L power:+3V3 #PWR?
+L power:+3V3 #PWR0102
 U 1 1 5B6756B8
 P 3150 6700
-F 0 "#PWR?" H 3150 6550 50  0001 C CNN
+F 0 "#PWR0102" H 3150 6550 50  0001 C CNN
 F 1 "+3V3" H 3150 6840 50  0000 C CNN
 F 2 "" H 3150 6700 50  0001 C CNN
