File: blackBoxProbeSmall/blackBoxProbeSmall.sch (KiCad schematic (older format))
At the start: 84 parts, among them J1 USB-ID, J2 JTAG_2X05, J3 JTAG_2X05, J4 Conn_01x04, Q1 Q_NMOS_DUAL, Q2 Q_PMOS_DUAL, U1 MCP1702-MB, U2 USBLC6-2, U3 STM32F103CBT, U4 74X2T45, U5 74X2T45, U6 74X2T45, U7 74X2T45, Y1 8.000MHz

Commit message: replaced all R's C's and inserted new box outline
Parts:
- removed R2, R3: R, SquantorRcl:R_0603_hand, symbol Device:R
- C10, C11, C12, C13, C15, C16, C17, C18, C19, C20, C21, C22, C3, C5, C6, C7, C8: footprint SquantorRcl:C_0603 -> SquantorRcl:C_0402
- J3: footprint SquantorConnectors:Header-Shr-0127-2X05-H006 -> SquantorConnectors:Header-0127-2X05-H006
- R1, R10, R11, R12, R13, R14, R15, R16, R17, R18, R19, R20, R21, R22, R23, R24, R25, R26, R27, R28, R29, R30, R31, R32, R33, R34, R35, R36, R37, R38, R4, R5, R6, R7, R8, R9: footprint SquantorRcl:R_0603_hand -> SquantorRcl:R_0402_hand
- U1: footprint SquantorMicrochip:MB-(SOT-89) -> SquantorIC:SOT89-ViaTab-Microchip-MB
Connections:
- wire segments 306 -> 300
- no-connect marks 9 -> 10
