File: blackBoxProbeSmall/blackBoxProbeSmall.sch (KiCad schematic (older format))
At the start: 78 parts, among them J1 USB-ID, J2 JTAG_2X05, J3 JTAG_2X05, J4 Conn_01x04, Q1 Q_NMOS_DUAL, Q2 Q_PMOS_DUAL, U1 MCP1702-MB, U2 USBLC6-2, U3 STM32F103CBT, U4 74X2T45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

Commit message: schematic conversion done, started placement of components
Parts:
- D1, D2, D3, D4: footprint LEDs:LED_D3.0mm -> LED_SMD:LED_0805_2012Metric_Castellated
- J3: footprint SquantorConnectors:Header-Shr-0127-2X05-H006 -> SquantorConnectors:Header-0127-2X05-H006
- J4: footprint Pin_Headers:Pin_Header_Angled_1x04_Pitch2.54mm -> Connector_JST:JST_PH_B4B-PH-SM4-TB_1x04-1MP_P2.00mm_Vertical
Changed lines of the file:
@@
 F 0 "J3" H 10000 1650 60  0000 C CNN
 F 1 "JTAG_2X05" H 10000 950 60  0000 C CNN
-F 2 "SquantorConnectors:Header-Shr-0127-2X05-H006" H 10000 1450 60  0001 C CNN
+F 2 "SquantorConnectors:Header-0127-2X05-H006" H 10000 1450 60  0001 C CNN
 F 3 "" H 10000 1450 60  0001 C CNN
 	1    10000 1300
@@
 F 0 "D1" H 950 6000 50  0000 C CNN
 F 1 "Green" H 950 5800 50  0000 C CNN
-F 2 "LEDs:LED_D3.0mm" H 950 5900 50  0001 C CNN
+F 2 "LED_SMD:LED_0805_2012Metric_Castellated" H 950 5900 50  0001 C CNN
 F 3 "" H 950 5900 50  0001 C CNN
 	1    950  5900
@@
 F 0 "D2" H 950 6300 50  0000 C CNN
 F 1 "Yellow" H 950 6100 50  0000 C CNN
-F 2 "LEDs:LED_D3.0mm" H 950 6200 50  0001 C CNN
+F 2 "LED_SMD:LED_0805_2012Metric_Castellated" H 950 6200 50  0001 C CNN
 F 3 "" H 950 6200 50  0001 C CNN
 	1    950  6200
@@
 F 0 "D3" H 950 6600 50  0000 C CNN
 F 1 "Orange" H 950 6400 50  0000 C CNN
-F 2 "LEDs:LED_D3.0mm" H 950 6500 50  0001 C CNN
+F 2 "LED_SMD:LED_0805_2012Metric_Castellated" H 950 6500 50  0001 C CNN
 F 3 "" H 950 6500 50  0001 C CNN
 	1    950  6500
@@
 F 0 "D4" H 950 6900 50  0000 C CNN
 F 1 "Red" H 950 6700 50  0000 C CNN
-F 2 "LEDs:LED_D3.0mm" H 950 6800 50  0001 C CNN
+F 2 "LED_SMD:LED_0805_2012Metric_Castellated" H 950 6800 50  0001 C CNN
 F 3 "" H 950 6800 50  0001 C CNN
 	1    950  6800
@@
 F 0 "J4" H 11050 2250 50  0000 C CNN
 F 1 "Conn_01x04" H 11050 1750 50  0000 C CNN
-F 2 "Pin_Headers:Pin_Header_Angled_1x04_Pitch2.54mm" H 11050 2050 50  0001 C CNN
+F 2 "Connector_JST:JST_PH_B4B-PH-SM4-TB_1x04-1MP_P2.00mm_Vertical" H 11050 2050 50  0001 C CNN
 F 3 "" H 11050 2050 50  0001 C CNN
 	1    11050 2050

Commit message: small updates in placement
Parts:
- C1: value 2.2u -> 1u; footprint SquantorRcl:C_0805 -> SquantorRcl:C_0603
Changed lines of the file:
@@
 EESchema Schematic File Version 4
+LIBS:blackBoxProbeSmall-cache
 EELAYER 26 0
 EELAYER END
@@
 P 750 1250
 F 0 "C1" H 775 1350 50  0000 L CNN
-F 1 "2.2u" H 775 1150 50  0000 L CNN
-F 2 "SquantorRcl:C_0805" H 788 1100 50  0001 C CNN
+F 1 "1u" H 775 1150 50  0000 L CNN
+F 2 "SquantorRcl:C_0603" H 788 1100 50  0001 C CNN
 F 3 "" H 750 1250 50  0001 C CNN
 	1    750  1250

Commit message: further placement of components, everything fits on pcb, now compacting due to smaller footprints
Parts:
- removed D1: Green, LED_SMD:LED_0805_2012Metric_Castellated, symbol Device:LED
- removed D2: Yellow, LED_SMD:LED_0805_2012Metric_Castellated, symbol Device:LED
- removed D3: Orange, LED_SMD:LED_0805_2012Metric_Castellated, symbol Device:LED
- removed D4: Red, LED_SMD:LED_0805_2012Metric_Castellated, symbol Device:LED
- removed N3: BlackBoxProbe, SquantorLabels:Label_version, symbol SquantorLabels:VYYYYMMDD
- added DA1: mentor_1296.4124, SquantorOpto:mentor_1296.4124, symbol SquantorOpto:mentor_1296.4124
- J4: footprint Connector_JST:JST_PH_B4B-PH-SM4-TB_1x04-1MP_P2.00mm_Vertical -> Connector_JST:JST_PH_S4B-PH-K_1x04_P2.00mm_Horizontal
Connections:
- wire segments 295 -> 300
Changed lines of the file:
@@
 PROBE_TMS_DIR
-$Comp
-L Device:Crystal Y1
-U 1 1 5B21AA36
-P 5550 6200
-F 0 "Y1" H 5550 6350 50  0000 C CNN
-F 1 "8.000MHz" H 5550 6050 50  0000 C CNN
-F 2 "SquantorCrystal:X_5.0_3.2" H 5550 6200 50  0001 C CNN
-F 3 "" H 5550 6200 50  0001 C CNN
-	1    5550 6200
-	0    1    1    0
-$EndComp
 $Comp
 L Device:C C12
@@
 L power:+3V3 #PWR079
 U 1 1 5B25622F
-P 1500 5900
-F 0 "#PWR079" H 1500 5750 50  0001 C CNN
-F 1 "+3V3" H 1500 6040 50  0000 C CNN
-F 2 "" H 1500 5900 50  0001 C CNN
-F 3 "" H 1500 5900 50  0001 C CNN
-	1    1500 5900
+P 2850 5950
+F 0 "#PWR079" H 2850 5800 50  0001 C CNN
+F 1 "+3V3" H 2850 6090 50  0000 C CNN
+F 2 "" H 2850 5950 50  0001 C CNN
+F 3 "" H 2850 5950 50  0001 C CNN
+	1    2850 5950
 	0    1    1    0
 $EndComp
@@
 L Device:R R29
 U 1 1 5B25639D
-P 1300 5900
-F 0 "R29" V 1380 5900 50  0000 C CNN
-F 1 "330" V 1300 5900 50  0000 C CNN
-F 2 "SquantorRcl:R_0402_hand" V 1230 5900 50  0001 C CNN
-F 3 "" H 1300 5900 50  0001 C CNN
-	1    1300 5900
-	0    -1   -1   0
-$EndComp
-$Comp
-L Device:LED D1
-U 1 1 5B256795
-P 950 5900
-F 0 "D1" H 950 6000 50  0000 C CNN
-F 1 "Green" H 950 5800 50  0000 C CNN
-F 2 "LED_SMD:LED_0805_2012Metric_Castellated" H 950 5900 50  0001 C CNN
-F 3 "" H 950 5900 50  0001 C CNN
-	1    950  5900
-	1    0    0    -1
+P 2600 5950
+F 0 "R29" V 2650 5750 50  0000 C CNN
+F 1 "330" V 2600 5950 50  0000 C CNN
+F 2 "SquantorRcl:R_0402_hand" V 2530 5950 50  0001 C CNN
+F 3 "" H 2600 5950 50  0001 C CNN
+	1    2600 5950
+	0    -1   -1   0
 $EndComp
 $Comp
 L power:GND #PWR080
 U 1 1 5B256978
-P 750 5900
-F 0 "#PWR080" H 750 5650 50  0001 C CNN
-F 1 "GND" H 750 5750 50  0000 C CNN
-F 2 "" H 750 5900 50  0001 C CNN
-F 3 "" H 750 5900 50  0001 C CNN
-	1    750  5900
-	0    1    1    0
-$EndComp
-Wire Wire Line
-	750  5900 800  5900
-Wire Wire Line
-	1100 5900 1150 5900
-Wire Wire Line
-	1450 5900 1500 5900
+P 1700 6100
+F 0 "#PWR080" H 1700 5850 50  0001 C CNN
+F 1 "GND" H 1700 5950 50  0000 C CNN
+F 2 "" H 1700 6100 50  0001 C CNN
+F 3 "" H 1700 6100 50  0001 C CNN
+	1    1700 6100
+	0    1    1    0
+$EndComp
+Wire Wire Line
+	1700 6100 1750 6100
+Wire Wire Line
+	2750 5950 2850 5950
 $Comp
 L Device:R R30
 U 1 1 5B257198
-P 1300 6200
-F 0 "R30" V 1380 6200 50  0000 C CNN
-F 1 "330" V 1300 6200 50  0000 C CNN
-F 2 "SquantorRcl:R_0402_hand" V 1230 6200 50  0001 C CNN
-F 3 "" H 1300 6200 50  0001 C CNN
-	1    1300 6200
-	0    -1   -1   0
-$EndComp
-$Comp
-L Device:LED D2
-U 1 1 5B25719E
-P 950 6200
-F 0 "D2" H 950 6300 50  0000 C CNN
-F 1 "Yellow" H 950 6100 50  0000 C CNN
-F 2 "LED_SMD:LED_0805_2012Metric_Castellated" H 950 6200 50  0001 C CNN
-F 3 "" H 950 6200 50  0001 C CNN
-	1    950  6200
-	1    0    0    -1
-$EndComp
-$Comp
-L power:GND #PWR081
-U 1 1 5B2571A4
-P 750 6200
-F 0 "#PWR081" H 750 5950 50  0001 C CNN
-F 1 "GND" H 750 6050 50  0000 C CNN
-F 2 "" H 750 6200 50  0001 C CNN
-F 3 "" H 750 6200 50  0001 C CNN
-	1    750  6200
-	0    1    1    0
-$EndComp
-Wire Wire Line
-	750  6200 800  6200
-Wire Wire Line
-	1100 6200 1150 6200
-Wire Wire Line
-	1450 6200 1500 6200
+P 2600 6050
+F 0 "R30" V 2650 5850 50  0000 C CNN
+F 1 "330" V 2600 6050 50  0000 C CNN
+F 2 "SquantorRcl:R_0402_hand" V 2530 6050 50  0001 C CNN
+F 3 "" H 2600 6050 50  0001 C CNN
+	1    2600 6050
+	0    -1   -1   0
+$EndComp
+Wire Wire Line
+	2400 6050 2450 6050
+Wire Wire Line
+	2750 6050 2900 6050
 $Comp
 L Device:R R31
 U 1 1 5B257543
-P 1300 6500
-F 0 "R31" V 1380 6500 50  0000 C CNN
-F 1 "330" V 1300 6500 50  0000 C CNN
-F 2 "SquantorRcl:R_0402_hand" V 1230 6500 50  0001 C CNN
-F 3 "" H 1300 6500 50  0001 C CNN
-	1    1300 6500
-	0    -1   -1   0
-$EndComp
-$Comp
-L Device:LED D3
-U 1 1 5B257549
-P 950 6500
-F 0 "D3" H 950 6600 50  0000 C CNN
-F 1 "Orange" H 950 6400 50  0000 C CNN
-F 2 "LED_SMD:LED_0805_2012Metric_Castellated" H 950 6500 50  0001 C CNN
-F 3 "" H 950 6500 50  0001 C CNN
-	1    950  6500
-	1    0    0    -1
-$EndComp
-$Comp
-L power:GND #PWR082
-U 1 1 5B25754F
-P 750 6500
-F 0 "#PWR082" H 750 6250 50  0001 C CNN
-F 1 "GND" H 750 6350 50  0000 C CNN
-F 2 "" H 750 6500 50  0001 C CNN
-F 3 "" H 750 6500 50  0001 C CNN
-	1    750  6500
-	0    1    1    0
-$EndComp
-Wire Wire Line
-	750  6500 800  6500
-Wire Wire Line
-	1100 6500 1150 6500
-Wire Wire Line
-	1450 6500 1500 6500
+P 2600 6150
+F 0 "R31" V 2650 5950 50  0000 C CNN
+F 1 "330" V 2600 6150 50  0000 C CNN
+F 2 "SquantorRcl:R_0402_hand" V 2530 6150 50  0001 C CNN
+F 3 "" H 2600 6150 50  0001 C CNN
+	1    2600 6150
+	0    -1   -1   0
+$EndComp
+Wire Wire Line
+	2400 6150 2450 6150
+Wire Wire Line
+	2750 6150 2900 6150
 $Comp
 L Device:R R32
 U 1 1 5B2576B0
-P 1300 6800
-F 0 "R32" V 1380 6800 50  0000 C CNN
-F 1 "330" V 1300 6800 50  0000 C CNN
-F 2 "SquantorRcl:R_0402_hand" V 1230 6800 50  0001 C CNN
-F 3 "" H 1300 6800 50  0001 C CNN
-	1    1300 6800
-	0    -1   -1   0
-$EndComp
-$Comp
-L Device:LED D4
-U 1 1 5B2576B6
-P 950 6800
-F 0 "D4" H 950 6900 50  0000 C CNN
-F 1 "Red" H 950 6700 50  0000 C CNN
-F 2 "LED_SMD:LED_0805_2012Metric_Castellated" H 950 6800 50  0001 C CNN
-F 3 "" H 950 6800 50  0001 C CNN
-	1    950  6800
-	1    0    0    -1
-$EndComp
-$Comp
-L power:GND #PWR083
-U 1 1 5B2576BC
-P 750 6800
-F 0 "#PWR083" H 750 6550 50  0001 C CNN
-F 1 "GND" H 750 6650 50  0000 C CNN
-F 2 "" H 750 6800 50  0001 C CNN
-F 3 "" H 750 6800 50  0001 C CNN
-	1    750  6800
-	0    1    1    0
-$EndComp
-Wire Wire Line
-	750  6800 800  6800
-Wire Wire Line
-	1100 6800 1150 6800
-Wire Wire Line
-	1450 6800 1500 6800
-Text Label 1500 6200 0    60   ~ 0
+P 2600 6250
+F 0 "R32" V 2650 6050 50  0000 C CNN
+F 1 "330" V 2600 6250 50  0000 C CNN
+F 2 "SquantorRcl:R_0402_hand" V 2530 6250 50  0001 C CNN
+F 3 "" H 2600 6250 50  0001 C CNN
+	1    2600 6250
+	0    -1   -1   0
+$EndComp
+Wire Wire Line
+	2400 6250 2450 6250
+Wire Wire Line
+	2750 6250 2900 6250
+Text Label 2900 6050 0    60   ~ 0
 LED0
-Text Label 1500 6500 0    60   ~ 0
+Text Label 2900 6150 0    60   ~ 0
 LED1
-Text Label 1500 6800 0    60   ~ 0
+Text Label 2900 6250 0    60   ~ 0
 LED2
 NoConn ~ 5950 5350
@@
 F 0 "J4" H 11050 2250 50  0000 C CNN
 F 1 "Conn_01x04" H 11050 1750 50  0000 C CNN
-F 2 "Connector_JST:JST_PH_B4B-PH-SM4-TB_1x04-1MP_P2.00mm_Vertical" H 11050 2050 50  0001 C CNN
+F 2 "Connector_JST:JST_PH_S4B-PH-K_1x04_P2.00mm_Horizontal" H 11050 2050 50  0001 C CNN
 F 3 "" H 11050 2050 50  0001 C CNN
 	1    11050 2050
@@
 Wire Wire Line
 	3400 3200 3450 3200
-$Comp
-L SquantorLabels:VYYYYMMDD N3
-U 1 1 5B31581F
-P 850 7500
-F 0 "N3" H 850 7600 60  0000 C CNN
-F 1 "BlackBoxProbe" H 850 7500 60  0000 C CNN
-F 2 "SquantorLabels:Label_version" H 850 7500 60  0001 C CNN
-F 3 "" H 850 7500 60  0001 C CNN
-	1    850  7500
-	1    0    0    -1
-$EndComp
 Text Label 9000 850  2    60   ~ 0
 PROBE_E_VDD
@@
 	5550 6450 5350 6450
 Wire Wire Line
-	5550 6000 5850 6000
-Wire Wire Line
 	800  4600 800  4650
 Wire Wire Line
@@
 Wire Wire Line
 	4400 6950 4500 6950
+$Comp
+L SquantorOpto:mentor_1296.4124 DA1
+U 1 1 5C0D962C
+P 2100 6100
+F 0 "DA1" H 2100 5663 60  0000 C CNN
+F 1 "mentor_1296.4124" H 2100 5769 60  0000 C CNN
+F 2 "SquantorOpto:mentor_1296.4124" H 2000 6100 60  0001 C CNN
+F 3 "" H 2000 6100 60  0001 C CNN
+	1    2100 6100
+	-1   0    0    1
+$EndComp
+Wire Wire Line
+	1750 5950 1750 6050
+Wire Wire Line
+	1750 6250 1800 6250
+Connection ~ 1750 6100
+Wire Wire Line
+	1750 6100 1750 6150
+Wire Wire Line
+	1800 5950 1750 5950
+Wire Wire Line
+	1750 6050 1800 6050
+Connection ~ 1750 6050
+Wire Wire Line
+	1750 6050 1750 6100
+Wire Wire Line
+	1800 6150 1750 6150
+Connection ~ 1750 6150
+Wire Wire Line
+	1750 6150 1750 6250
+Wire Wire Line
+	2400 5950 2450 5950
+Wire Wire Line
+	5550 6000 5850 6000
+$Comp
+L Device:Crystal Y1
+U 1 1 5B21AA36
+P 5550 6200
+F 0 "Y1" H 5550 6350 50  0000 C CNN
+F 1 "8.000MHz" H 5550 6050 50  0000 C CNN
+F 2 "SquantorCrystal:X_5.0_3.2" H 5550 6200 50  0001 C CNN
+F 3 "" H 5550 6200 50  0001 C CNN
+	1    5550 6200
+	0    1    1    0
+$EndComp
 $EndSCHEMATC
