File: blackBoxProbeBig/blackBoxProbeBig.sch (KiCad schematic (older format))
At the start: 84 parts, among them J1 USB-ID, J2 JTAG_2X05, J3 JTAG_2X05, J4 Conn_01x04, Q1 Q_NMOS_DUAL, Q2 Q_PMOS_DUAL, U1 MCP1702-MB, U2 USBLC6-2, U3 STM32F103CBT, U4 74X2T45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

Commit message: footprint updates
Parts:
- U4, U5, U6, U7: footprint SquantorIC:NXP_SOT765-1_HAND -> SquantorIC:SOT765-1-NXP
Changed lines of the file:
@@
 EESchema Schematic File Version 4
-LIBS:blackBoxProbe-cache
+LIBS:blackBoxProbeBig-cache
 EELAYER 26 0
 EELAYER END
@@
 F 0 "U4" H 7100 1200 60  0000 C CNN
 F 1 "74X2T45" H 7100 600 60  0000 C CNN
-F 2 "SquantorIC:NXP_SOT765-1_HAND" H 7100 950 60  0001 C CNN
+F 2 "SquantorIC:SOT765-1-NXP" H 7100 950 60  0001 C CNN
 F 3 "" H 7100 950 60  0001 C CNN
 	1    7100 900
@@
 F 0 "U5" H 7100 1900 60  0000 C CNN
 F 1 "74X2T45" H 7100 1300 60  0000 C CNN
-F 2 "SquantorIC:NXP_SOT765-1_HAND" H 7100 1650 60  0001 C CNN
+F 2 "SquantorIC:SOT765-1-NXP" H 7100 1650 60  0001 C CNN
 F 3 "" H 7100 1650 60  0001 C CNN
 	1    7100 1600
@@
 F 0 "U6" H 7100 2600 60  0000 C CNN
 F 1 "74X2T45" H 7100 2000 60  0000 C CNN
-F 2 "SquantorIC:NXP_SOT765-1_HAND" H 7100 2350 60  0001 C CNN
+F 2 "SquantorIC:SOT765-1-NXP" H 7100 2350 60  0001 C CNN
 F 3 "" H 7100 2350 60  0001 C CNN
 	1    7100 2300
@@
 F 0 "U7" H 7100 3300 60  0000 C CNN
 F 1 "74X2T45" H 7100 2700 60  0000 C CNN
-F 2 "SquantorIC:NXP_SOT765-1_HAND" H 7100 3050 60  0001 C CNN
+F 2 "SquantorIC:SOT765-1-NXP" H 7100 3050 60  0001 C CNN
 F 3 "" H 7100 3050 60  0001 C CNN
 	1    7100 3000

Commit message: simplified schematic to be more in line with black magic probe v2.1
Parts:
- removed R17: 1K, SquantorRcl:R_0603_hand, symbol Device:R
- removed R19: 10, SquantorRcl:R_0603_hand, symbol Device:R
- removed R2, R3: R, SquantorRcl:R_0603_hand, symbol Device:R
- removed R23: 10K, SquantorRcl:R_0603_hand, symbol Device:R
- R36: value 100 -> 22
Connections:
- net +3V3: now also J2.1 (VCC)
- net GND: now also J1.4 (ID), U3.44 (BOOT0)
- net PROBE_E_VDD: now also R20.1
- net PROBE_VDD: no longer R20.1
Other:
- moved on the sheet: C11, J4, R10, R11, R21, R22, R33, R35, R36

Commit message: updated versionnumber
Parts:
- N2: value V20180728 -> V20181130
Changed lines of the file:
@@
 P 850 7700
 F 0 "N2" H 850 7800 60  0000 C CNN
-F 1 "V20180728" H 850 7700 60  0000 C CNN
+F 1 "V20181130" H 850 7700 60  0000 C CNN
 F 2 "SquantorLabels:Label_version" H 850 7700 60  0001 C CNN
 F 3 "" H 850 7700 60  0001 C CNN

Commit message: updated regulator with via variant
Parts:
- U1: footprint SquantorMicrochip:MB-(SOT-89) -> SquantorIC:SOT89-ViaTab-Microchip-MB
Changed lines of the file:
@@
 EESchema Schematic File Version 4
-LIBS:blackBoxProbeBig-cache
 EELAYER 26 0
 EELAYER END
@@
 F 0 "U1" H 1200 1500 60  0000 C CNN
 F 1 "MCP1702-MB" H 1200 1000 60  0000 C CNN
-F 2 "SquantorMicrochip:MB-(SOT-89)" H 1200 1250 60  0001 C CNN
+F 2 "SquantorIC:SOT89-ViaTab-Microchip-MB" H 1200 1250 60  0001 C CNN
 F 3 "" H 1200 1250 60  0001 C CNN
 	1    1200 1250

Commit message: schematic simplifications, regulator rework, silk movements
Parts:
- removed C3: 100n, SquantorRcl:C_0603, symbol Device:C
Other:
- moved on the sheet: C1
Changed lines of the file:
@@
 L Device:C C1
 U 1 1 5ABDD0E1
-P 1150 2450
-F 0 "C1" H 1175 2550 50  0000 L CNN
-F 1 "2.2u" H 1175 2350 50  0000 L CNN
-F 2 "SquantorRcl:C_0805" H 1188 2300 50  0001 C CNN
-F 3 "" H 1150 2450 50  0001 C CNN
-	1    1150 2450
-	1    0    0    -1
-$EndComp
-$Comp
-L power:+5V #PWR04
-U 1 1 5ABDD188
-P 1150 2250
-F 0 "#PWR04" H 1150 2100 50  0001 C CNN
-F 1 "+5V" H 1150 2390 50  0000 C CNN
-F 2 "" H 1150 2250 50  0001 C CNN
-F 3 "" H 1150 2250 50  0001 C CNN
-	1    1150 2250
-	1    0    0    -1
-$EndComp
-$Comp
-L power:GND #PWR05
-U 1 1 5ABDD217
-P 1150 2650
-F 0 "#PWR05" H 1150 2400 50  0001 C CNN
-F 1 "GND" H 1150 2500 50  0000 C CNN
-F 2 "" H 1150 2650 50  0001 C CNN
-F 3 "" H 1150 2650 50  0001 C CNN
-	1    1150 2650
+P 750 1250
+F 0 "C1" H 775 1350 50  0000 L CNN
+F 1 "2.2u" H 775 1150 50  0000 L CNN
+F 2 "SquantorRcl:C_0805" H 788 1100 50  0001 C CNN
+F 3 "" H 750 1250 50  0001 C CNN
+	1    750  1250
 	1    0    0    -1
 $EndComp
@@
 	1    1300 1600
 	-1   0    0    1
-$EndComp
-$Comp
-L Device:C C3
-U 1 1 5ABDED68
-P 750 1250
-F 0 "C3" H 775 1350 50  0000 L CNN
-F 1 "100n" H 775 1150 50  0000 L CNN
-F 2 "SquantorRcl:C_0603" H 788 1100 50  0001 C CNN
-F 3 "" H 750 1250 50  0001 C CNN
-	1    750  1250
-	1    0    0    -1
 $EndComp
 $Comp
@@
 	1450 3050 1800 3050
 Wire Wire Line
-	1150 2300 1150 2250
-Wire Wire Line
-	1150 2600 1150 2650
-Wire Wire Line
 	1200 1800 1200 1550

Commit message: updated component footprints
Parts:
- C1: value 2.2u -> 1u; footprint SquantorRcl:C_0805 -> SquantorRcl:C_0603
Changed lines of the file:
@@
 EESchema Schematic File Version 4
+LIBS:blackBoxProbeBig-cache
 EELAYER 26 0
 EELAYER END
@@
 P 750 1250
 F 0 "C1" H 775 1350 50  0000 L CNN
-F 1 "2.2u" H 775 1150 50  0000 L CNN
-F 2 "SquantorRcl:C_0805" H 788 1100 50  0001 C CNN
+F 1 "1u" H 775 1150 50  0000 L CNN
+F 2 "SquantorRcl:C_0603" H 788 1100 50  0001 C CNN
 F 3 "" H 750 1250 50  0001 C CNN
 	1    750  1250
