File: electronics/blackBoxProbeMicro/blackBoxProbeMicro.kicad_sch (KiCad schematic)
At the start: 66 parts, among them J1 USB-C, J2 JTAG_2X05, J3 JTAG_2X05, J4 DevBoardUartOutput, Q1 BSD840N, Q2 NTJD4152P, U1 MCP1702-MB, U2 DT1446-04S, U3 STM32F103CBT, Y1 8MHz

Commit message: prepared for production
Parts:
- N2: value V:20240216 -> V:20240218
Changed lines of the file:
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@@
       (effects (font (size 1.524 1.524)))
     )
-    (property "Value" "V:20240216" (at 24.13 181.61 0)
+    (property "Value" "V:20240218" (at 24.13 181.61 0)
       (effects (font (size 1.524 1.524)))
     )
